Commit message: modify
Signed-off-by: Yamato Ando <yamato.ando@gmail.com>

File: src/vehicle/util/vehicle_launch/urdf/vehicle.xacro (robot description, xacro)
@@ -8,5 +8,5 @@
   <xacro:include filename="$(find camera_description)/urdf/monocular_camera.xacro"/>
   <xacro:include filename="$(find imu_description)/urdf/imu.xacro"/>
-  <xacro:property name="calibration" value="${load_yaml('$(find vehicle_launch)/vehicle_description/config/calibration.yaml')}"/>
+  <xacro:property name="calibration" value="${load_yaml('$(find vehicle_launch)/config/calibration.yaml')}"/>
   <xacro:arg name="gpu" default="false"/>
   <!-- lidar -->
