Commit message: fix sensor calib
Signed-off-by: Yamato Ando <yamato.ando@gmail.com>

File: src/launcher/vehicle_launch/urdf/vehicle.xacro (robot description, xacro)
@@ -1,34 +1,10 @@
 <?xml version="1.0"?>
-<robot name="vehicle" xmlns:xacro="http://ros.org/wiki/xacro">
-  <!-- vehicle -->
+<robot name="vehicle"
+  xmlns:xacro="http://ros.org/wiki/xacro">
   <xacro:include filename="$(find lexus_description)/urdf/lexus.xacro"/>
-  <!-- sensor -->
-  <xacro:include filename="$(find velodyne_description)/urdf/HDL-32E.urdf.xacro"/>
-  <xacro:include filename="$(find velodyne_description)/urdf/VLP-16.urdf.xacro"/>
-  <xacro:include filename="$(find camera_description)/urdf/monocular_camera.xacro"/>
-  <xacro:include filename="$(find imu_description)/urdf/imu.xacro"/>
-  <xacro:property name="calibration" value="${load_yaml('$(find vehicle_launch)/config/calibration.yaml')}"/>
-  <xacro:arg name="gpu" default="false"/>
-  <!-- lidar -->
-  <VLP-16 parent="base_link" name="velodyne_top" topic="/points_raw" hz="10" samples="220" gpu="$(arg gpu)">
-    <origin xyz="${calibration['base_link2velodyne_top']['x']} ${calibration['base_link2velodyne_top']['y']} ${calibration['base_link2velodyne_top']['z']}" rpy="${calibration['base_link2velodyne_top']['roll']} ${calibration['base_link2velodyne_top']['pitch']} ${calibration['base_link2velodyne_top']['yaw']}" />
-  </VLP-16>
-  <VLP-16 parent="base_link" name="velodyne_left" topic="/points_raw" hz="10" samples="220" gpu="$(arg gpu)">
-    <origin xyz="${calibration['base_link2velodyne_left']['x']} ${calibration['base_link2velodyne_left']['y']} ${calibration['base_link2velodyne_left']['z']}" rpy="${calibration['base_link2velodyne_left']['roll']} ${calibration['base_link2velodyne_left']['pitch']} ${calibration['base_link2velodyne_left']['yaw']}" />
-  </VLP-16>
-  <VLP-16 parent="base_link" name="velodyne_right" topic="/points_raw" hz="10" samples="220" gpu="$(arg gpu)">
-    <origin xyz="${calibration['base_link2velodyne_right']['x']} ${calibration['base_link2velodyne_right']['y']} ${calibration['base_link2velodyne_right']['z']}" rpy="${calibration['base_link2velodyne_right']['roll']} ${calibration['base_link2velodyne_right']['pitch']} ${calibration['base_link2velodyne_right']['yaw']}" />
-  </VLP-16>
-  <!-- camera -->
-  <xacro:monocular_camera_macro suffix="traffic_light/camera" parent="base_link" namespace="" x="${calibration['base_link2traffic_light_camera']['x']}" y="${calibration['base_link2traffic_light_camera']['y']}" z="${calibration['base_link2traffic_light_camera']['z']}" roll="${calibration['base_link2traffic_light_camera']['roll']}" pitch="${calibration['base_link2traffic_light_camera']['pitch']}" yaw="${calibration['base_link2traffic_light_camera']['yaw']}" fps="30" width="800" height="400" fov="1.3"/>
-  <xacro:monocular_camera_macro suffix="camera1/camera" parent="base_link" namespace="" x="${calibration['base_link2camera1']['x']}" y="${calibration['base_link2camera1']['y']}" z="${calibration['base_link2camera1']['z']}" roll="${calibration['base_link2camera1']['roll']}" pitch="${calibration['base_link2camera1']['pitch']}" yaw="${calibration['base_link2camera1']['yaw']}" fps="30" width="800" height="400" fov="1.3"/>
-  <xacro:monocular_camera_macro suffix="camera2/camera" parent="base_link" namespace="" x="${calibration['base_link2camera2']['x']}" y="${calibration['base_link2camera2']['y']}" z="${calibration['base_link2camera2']['z']}" roll="${calibration['base_link2camera2']['roll']}" pitch="${calibration['base_link2camera2']['pitch']}" yaw="${calibration['base_link2camera2']['yaw']}" fps="30" width="800" height="400" fov="1.3"/>
-  <xacro:monocular_camera_macro suffix="camera3/camera" parent="base_link" namespace="" x="${calibration['base_link2camera3']['x']}" y="${calibration['base_link2camera3']['y']}" z="${calibration['base_link2camera3']['z']}" roll="${calibration['base_link2camera3']['roll']}" pitch="${calibration['base_link2camera3']['pitch']}" yaw="${calibration['base_link2camera3']['yaw']}" fps="30" width="800" height="400" fov="1.3"/>
-  <xacro:monocular_camera_macro suffix="camera4/camera" parent="base_link" namespace="" x="${calibration['base_link2camera4']['x']}" y="${calibration['base_link2camera4']['y']}" z="${calibration['base_link2camera4']['z']}" roll="${calibration['base_link2camera4']['roll']}" pitch="${calibration['base_link2camera4']['pitch']}" yaw="${calibration['base_link2camera4']['yaw']}" fps="30" width="800" height="400" fov="1.3"/>
-  <xacro:monocular_camera_macro suffix="camera5/camera" parent="base_link" namespace="" x="${calibration['base_link2camera5']['x']}" y="${calibration['base_link2camera5']['y']}" z="${calibration['base_link2camera5']['z']}" roll="${calibration['base_link2camera5']['roll']}" pitch="${calibration['base_link2camera5']['pitch']}" yaw="${calibration['base_link2camera5']['yaw']}" fps="30" width="800" height="400" fov="1.3"/>
-  <xacro:monocular_camera_macro suffix="camera6/camera" parent="base_link" namespace="" x="${calibration['base_link2camera6']['x']}" y="${calibration['base_link2camera6']['y']}" z="${calibration['base_link2camera6']['z']}" roll="${calibration['base_link2camera6']['roll']}" pitch="${calibration['base_link2camera6']['pitch']}" yaw="${calibration['base_link2camera6']['yaw']}" fps="30" width="800" height="400" fov="1.3"/>
-  <!-- imu -->
-  <xacro:imu_macro suffix="gx5/imu" parent="base_link" namespace="" x="${calibration['base_link2imu_gx5']['x']}" y="${calibration['base_link2imu_gx5']['y']}" z="${calibration['base_link2imu_gx5']['z']}" roll="${calibration['base_link2imu_gx5']['roll']}" pitch="${calibration['base_link2imu_gx5']['pitch']}" yaw="${calibration['base_link2imu_gx5']['yaw']}" fps="100" />
-  <xacro:imu_macro suffix="tamagawa/imu" parent="base_link" namespace="" x="${calibration['base_link2imu_tamagawa']['x']}" y="${calibration['base_link2imu_tamagawa']['y']}" z="${calibration['base_link2imu_tamagawa']['z']}" roll="${calibration['base_link2imu_tamagawa']['roll']}" pitch="${calibration['base_link2imu_tamagawa']['pitch']}" yaw="${calibration['base_link2imu_tamagawa']['yaw']}" fps="100" />
+  <xacro:include filename="$(find vehicle_launch)/urdf/aipxx.xacro"/>
+  <xacro:property name="calibration" value="${load_yaml('$(find vehicle_launch)/config/sensors_calibration.yaml')}"/>
+  <!-- aipxx -->
+  <xacro:aipxx_macro parent="base_link" x="${calibration['base_link2aipxx_base_link']['x']}" y="${calibration['base_link2aipxx_base_link']['y']}" z="${calibration['base_link2aipxx_base_link']['z']}" roll="${calibration['base_link2aipxx_base_link']['roll']}" pitch="${calibration['base_link2aipxx_base_link']['pitch']}" yaw="${calibration['base_link2aipxx_base_link']['yaw']}" />
   <!-- gnss -->
   <xacro:imu_macro suffix="gnss" parent="base_link" namespace="" x="${calibration['base_link2gnss']['x']}" y="${calibration['base_link2gnss']['y']}" z="${calibration['base_link2gnss']['z']}" roll="${calibration['base_link2gnss']['roll']}" pitch="${calibration['base_link2gnss']['pitch']}" yaw="${calibration['base_link2gnss']['yaw']}" fps="100" />
